File: cp-test-project/cp-test-project.kicad_sch (KiCad schematic)
At the start: 0 parts

Commit message: rev-1 created
Other:
- note added: "rev-1"
- note removed: "MAIN"
Changed lines of the file:
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@@
 	(generator_version "8.0")
 	(paper "A4")
-	(text "MAIN"
+	(text "rev-1"
 		(exclude_from_sim no)
 		(at 140.716 80.772 0)

Commit message: rev-2
Other:
- added sheet sheet1 (sheet1-page.kicad_sch)
- note added: "rev-2"
- note removed: "rev-1"
Changed lines of the file:
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@@
 	(generator_version "8.0")
 	(paper "A4")
-	(text "rev-1"
+	(text "rev-2"
 		(exclude_from_sim no)
 		(at 140.716 80.772 0)
@@
 			)
 		)
+	)
+	(sheet
+		(at 68.58 106.68)
+		(size 58.42 49.53)
+		(fields_autoplaced yes)
+		(stroke
+			(width 0.1524)
+			(type solid)
+		)
+		(fill
+			(color 0 0 0 0.0000)
+		)
+		(property "Sheetname" "sheet1"
+			(at 68.58 105.9684 0)
+			(effects
+				(font
+					(size 1.27 1.27)
+				)
+				(justify left bottom)
+			)
+		)
+		(property "Sheetfile" "sheet1-page.kicad_sch"
+			(at 68.58 156.7946 0)
+			(effects
+				(font
+					(size 1.27 1.27)
+				)
+				(justify left top)
+			)
+		)
+		(instances
+			(project "cp-test-project"
+				(path "/396724f0-1018-470f-8cbe-43f9bf3e51d0"
+					(page "2")
+				)
+			)
+		)

Commit message: added tt
Other:
- added sheet tt (tt.kicad_sch)
Changed lines of the file:
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@@
+		)
+	)
+	(sheet
+		(at 190.5 116.84)
+		(size 38.1 3.81)
+		(fields_autoplaced yes)
+		(stroke
+			(width 0.1524)
+			(type solid)
+		)
+		(fill
+			(color 0 0 0 0.0000)
+		)
+		(property "Sheetname" "tt"
+			(at 190.5 116.1284 0)
+			(effects
+				(font
+					(size 1.27 1.27)
+				)
+				(justify left bottom)
+			)
+		)
+		(property "Sheetfile" "tt.kicad_sch"
+			(at 190.5 121.2346 0)
+			(effects
+				(font
+					(size 1.27 1.27)
+				)
+				(justify left top)
+			)
+		)
+		(instances
+			(project "cp-test-project"
+				(path "/396724f0-1018-470f-8cbe-43f9bf3e51d0"
+					(page "3")
+				)
+			)
 		)
 	)

Commit message: added t1
Other:
- added sheet t1 (t1.kicad_sch)
Changed lines of the file:
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@@
+	)
+	(sheet
+		(at 152.4 158.75)
+		(size 35.56 3.81)
+		(fields_autoplaced yes)
+		(stroke
+			(width 0.1524)
+			(type solid)
+		)
+		(fill
+			(color 0 0 0 0.0000)
+		)
+		(property "Sheetname" "t1"
+			(at 152.4 158.0384 0)
+			(effects
+				(font
+					(size 1.27 1.27)
+				)
+				(justify left bottom)
+			)
+		)
+		(property "Sheetfile" "t1.kicad_sch"
+			(at 152.4 163.1446 0)
+			(effects
+				(font
+					(size 1.27 1.27)
+				)
+				(justify left top)
+			)
+		)
+		(instances
+			(project "cp-test-project"
+				(path "/396724f0-1018-470f-8cbe-43f9bf3e51d0"
+					(page "4")
+				)
+			)
+		)
 	)
 	(sheet
